File: keyboard61.kicad_pcb (KiCad board)
At the start: 2 copper layers, 295 x 168 mm, 128 parts, among them SW1 Esc, SW10 9, SW11 0, SW12 -, SW13 =, SW14 Backspace, SW15 Tab, SW16 Q, SW17 W, SW18 E, SW19 R, SW2 1, SW20 T, SW21 Y, SW22 U, SW23 I, SW24 O, SW25 P, SW26 [, SW27 ], SW28 Backslash, SW29 Caps, SW3 2, SW30 A, SW31 S, SW32 D, SW33 F, SW34 G, SW35 H, SW36 J, SW37 K, SW38 L, SW39 ;, SW4 3, SW40 Quote, SW41 Enter, SW42 LShift, SW43 Z, SW44 X, SW45 C, SW46 V, SW47 B, SW48 N, SW49 M, SW5 4, SW50 ,, SW51 ., SW52 /, SW53 RShift, SW54 LCtrl, SW55 LWin, SW56 LAlt, SW57 Space, SW58 RAlt, SW59 Fn, SW6 5, SW60 Menu, SW61 RCtrl, SW62 RESET, SW7 6, SW8 7, SW9 8, U1 Raspberry Pi Pico

Commit message: BOM
Parts:
- SW15: footprint Button_Switch_Keyboard:SW_Cherry_MX_1.50u_PCB -> Keyboard61:SW_Cherry_MX_1.50u_PCB_SocketClearance
- SW16: footprint Button_Switch_Keyboard:SW_Cherry_MX_1.00u_PCB -> Keyboard61:SW_Cherry_MX_1.00u_PCB_SocketClearance
- SW62: moved to B.Cu
- U1: footprint Module:RaspberryPi_Pico_Common_THT -> Keyboard61:Pico_H_Bottom_Sockets_8_5mm; moved to B.Cu
- moved U1 157.1 mm to (48.3, 133.4), turned to -90 degrees
- moved D15 144.7 mm to (200.0, 211.5)
- moved SW62 144.5 mm to (335.0, 180.0), turned to 180 degrees
- moved D16 134.9 mm to (213.0, 211.5)
- moved D17 129.5 mm to (226.0, 211.5)
- moved D1 111.1 mm to (142.0, 211.5)
- moved D2 106.9 mm to (155.0, 211.5)
- moved D3 102.9 mm to (168.0, 211.5)
- moved H1 68.0 mm to (49.0, 117.0)
- moved H2 68.0 mm to (336.0, 117.0)
Routing:
- net GND: track 121.4 -> 371.0 mm, vias 0 -> 1
- net RUN: track 35.8 -> 273.2 mm
- net Net-(D15-A): track 16.3 -> 184.1 mm, vias 0 -> 1
- net Net-(D16-A): track 16.4 -> 175.7 mm, vias 0 -> 1
- net COL0: track 253.9 -> 94.7 mm
- net Net-(D17-A): track 16.4 -> 155.5 mm, vias 0 -> 2
- net Net-(D1-A): track 16.3 -> 153.5 mm
- net COL1: track 227.2 -> 108.0 mm
- net COL12: track 154.3 -> 268.0 mm, vias 0 -> 1
- net COL13: track 148.2 -> 256.8 mm
- net COL11: track 161.9 -> 270.3 mm, vias 0 -> 1
- net Net-(D2-A): track 22.1 -> 128.4 mm
- net COL10: track 146.5 -> 246.0 mm
- net Net-(D3-A): track 22.0 -> 120.3 mm
- net COL8: track 118.0 -> 208.0 mm
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Other:
- board size 295 x 168 mm -> 295 x 100 mm
- board text added: "PICO UNDER PCB / 8.5mm SOCKETS"
- board text added: "USB <"
- board text removed: "2 LAYERS / 1.6 mm FR4"
- board text removed: "61-KEY ANSI / RP2040"
- board text removed: "ASSEMBLY: DIODE STRIPE TO K PAD"
- board text removed: "DIODES: BACK / K = STRIPE"
- board text removed: "GPIO0-4 ROW / GPIO5-18 COL"
- board text removed: "KEYBOARD61"
- board text removed: "MX SWITCHES: FRONT"
- board text removed: "REV 1.0 | 2026-10-06"
- board text removed: "USB ON PICO"

Commit message: BOM
Parts:
- moved U1 51.4 mm to (96.6, 151.2), turned to 90 degrees
Routing:
- net COL9: track 208.3 -> 273.1 mm, vias 1 -> 0
- net ROW1: track 396.0 -> 335.3 mm, vias 2 -> 0
- net COL6: track 276.2 -> 329.5 mm
- net COL11: track 270.3 -> 321.2 mm, vias 1 -> 0
- net COL10: track 246.0 -> 291.0 mm, vias 1 -> 0
- net COL12: track 268.0 -> 305.7 mm, vias 1 -> 0
- net ROW0: track 413.9 -> 380.3 mm
- net COL13: track 256.8 -> 287.2 mm
- net ROW4: track 367.2 -> 338.0 mm
- net COL8: track 208.0 -> 233.6 mm, vias 0 -> 1
- net ROW2: track 310.0 -> 285.0 mm
- net RUN: track 273.2 -> 294.1 mm, vias 0 -> 1
- net ROW3: track 319.6 -> 299.2 mm
- net COL0: track 94.7 -> 114.2 mm, vias 1 -> 0
- net Net-(D17-A): track 155.5 -> 174.7 mm
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Other:
- board text added: "CASE POCKET / CABLE CHANNEL PLAN UNDER PCB - NO PCB CUTOUT MEASURE ACTUAL PLUG BEFORE CASE DESIGN"
- board text added: "USB > INWARD"
- board text removed: "USB <"

Commit message: BOM
Connections:
- U1 pad 25: unconnected-(U1-GPIO19-Pad25) -> ENC_A
- U1 pad 26: unconnected-(U1-GPIO20-Pad26) -> ENC_B
- U1 pad 27: unconnected-(U1-GPIO21-Pad27) -> ENC_SW
Changed lines of the file:
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@@
 			(layers "*.Cu" "*.Mask")
 			(remove_unused_layers no)
-			(net "unconnected-(U1-GPIO19-Pad25)")
+			(net "ENC_A")
 		)
 		(pad "26" thru_hole circle
@@
 			(layers "*.Cu" "*.Mask")
 			(remove_unused_layers no)
-			(net "unconnected-(U1-GPIO20-Pad26)")
+			(net "ENC_B")
 		)
 		(pad "27" thru_hole circle
@@
 			(layers "*.Cu" "*.Mask")
 			(remove_unused_layers no)
-			(net "unconnected-(U1-GPIO21-Pad27)")
+			(net "ENC_SW")
 		)
 		(pad "28" thru_hole custom

Commit message: BOM
Connections:
- U1 pad 29: unconnected-(U1-GPIO22-Pad29) -> TFT_DC
- U1 pad 31: unconnected-(U1-GPIO26_ADC0-Pad31) -> TFT_SCK
- U1 pad 32: unconnected-(U1-GPIO27_ADC1-Pad32) -> TFT_MOSI
- U1 pad 34: unconnected-(U1-GPIO28_ADC2-Pad34) -> TFT_CS
- U1 pad 36: unconnected-(U1-3V3-Pad36) -> 3V3
